Commit message: added ros2_control. modified launch file so that the user can specify whether to use ros2_control or not. set up controllers for ros2_control, and created separate ros_gz_bridge parameter files. changed friction parameters mu1 and mu2 so that the agent motion in rviz2 best reflects that of Gazebo

File: ros2_ws/src/agent_bringup/urdf/agent.urdf.xacro (robot description, xacro)
@@ -9,3 +9,11 @@
     <xacro:include filename = "agent_peripherals.xacro"/>
     <xacro:include filename = "agent_gazebo_properties.xacro"/>
+    <!-- if using ros2_control -->
+    <xacro:if value = "$(arg use_ros_control)">
+        <xacro:include filename = "agent_ros_control.xacro"/>
+    </xacro:if>
+    <!-- if using gazebo control -->
+    <xacro:unless value = "$(arg use_ros_control)">
+        <xacro:include filename = "agent_gazebo_control.xacro"/>
+    </xacro:unless>
 </robot>

File: ros2_ws/src/agent_bringup/urdf/agent_body.xacro (robot description, xacro)
@@ -85,6 +85,6 @@
             <origin xyz = "0 0 ${-o}" rpy = "1.570796 0 0"/>
             <geometry>
-                <cylinder radius = "0.0325" length = "0.03035"/>
-                <!-- <sphere radius = "0.0325"/> -->
+                <!-- <cylinder radius = "0.0325" length = "0.03035"/> -->
+                <sphere radius = "0.0325"/>
             </geometry>
         </collision>
@@ -119,6 +119,6 @@
             <origin xyz = "0 0 ${-o}" rpy = "1.570796 0 0"/>
             <geometry>
-                <cylinder radius = "0.0325" length = "0.03035"/>
-                <!-- <sphere radius = "0.0325"/> -->
+                <!-- <cylinder radius = "0.0325" length = "0.03035"/> -->
+                <sphere radius = "0.0325"/>
             </geometry>
         </collision>
@@ -153,6 +153,6 @@
             <origin xyz = "0 0 ${-o}" rpy = "1.570796 0 0"/>
             <geometry>
-                <cylinder radius = "0.0325" length = "0.03035"/>
-                <!-- <sphere radius = "0.0325"/> -->
+                <!-- <cylinder radius = "0.0325" length = "0.03035"/> -->
+                <sphere radius = "0.0325"/>
             </geometry>
         </collision>
@@ -187,6 +187,6 @@
             <origin xyz = "0 0 ${-o}" rpy = "1.570796 0 0"/>
             <geometry>
-                <cylinder radius = "0.0325" length = "0.03035"/>
-                <!-- <sphere radius = "0.0325"/> -->
+                <!-- <cylinder radius = "0.0325" length = "0.03035"/> -->
+                <sphere radius = "0.0325"/>
             </geometry>
         </collision>

File: ros2_ws/src/agent_bringup/urdf/agent_gazebo_properties.xacro (robot description, xacro)
@@ -2,6 +2,6 @@
 <robot xmlns:xacro = "http://www.ros.org/wiki/xacro">
     <!-- PROPERTIES -->
-    <xacro:property name = "mu1" value = "0.1"/>
-    <xacro:property name = "mu2" value = "0.1"/>
+    <xacro:property name = "mu1" value = "0.50"/>
+    <xacro:property name = "mu2" value = "0.01"/>
     <xacro:property name = "minDepth" value = "0.0001"/>
     <xacro:property name = "piValue" value = "3.14159265359"/>
@@ -10,4 +10,5 @@
         <mu1 value = "${mu1}"/>
         <mu2 value = "${mu2}"/>
+        <fdir1>1 0 0</fdir1>
         <minDepth value = "${minDepth}"/>
     </gazebo>
@@ -15,4 +16,5 @@
         <mu1 value = "${mu1}"/>
         <mu2 value = "${mu2}"/>
+        <fdir1>1 0 0</fdir1>
         <minDepth value = "${minDepth}"/>
     </gazebo>
@@ -20,4 +22,5 @@
         <mu1 value = "${mu1}"/>
         <mu2 value = "${mu2}"/>
+        <fdir1>1 0 0</fdir1>
         <minDepth value = "${minDepth}"/>
     </gazebo>
@@ -25,4 +28,5 @@
         <mu1 value = "${mu1}"/>
         <mu2 value = "${mu2}"/>
+        <fdir1>1 0 0</fdir1>
         <minDepth value = "${minDepth}"/>
     </gazebo>
@@ -55,43 +59,3 @@
         </sensor>
     </gazebo>
-    <xacro:unless value = "$(arg use_ros_control)">
-        <gazebo>
-            <!-- plugin for doing the control -->
-            <plugin name = "ignition::gazebo::systems::MecanumDrive" filename = "ignition-gazebo-mecanum-drive-system">
-                <!-- information about the robot -->
-                <front_left_joint>${prefix}_front_left_joint</front_left_joint>
-                <front_right_joint>${prefix}_front_right_joint</front_right_joint>
-                <back_left_joint>${prefix}_back_left_joint</back_left_joint>
-                <back_right_joint>${prefix}_back_right_joint</back_right_joint>
-                <wheelbase>0.16</wheelbase>
-                <wheel_separation>0.1695</wheel_separation>
-                <wheel_radius>0.0325</wheel_radius>
-                <!-- topic information -->
-                <odom_publish_frequency>60</odom_publish_frequency>
-                <topic>cmd_vel</topic>
-                <odom_topic>odom</odom_topic>
-                <tf_topic>tf</tf_topic>
-                <frame_id>odom</frame_id>
-                <child_frame_id>${prefix}_base_link</child_frame_id>
-            </plugin>
-            <!-- plugin for publishing odometry because the mecanum one cannot -->
-            <plugin name = "ignition::gazebo::systems::OdometryPublisher" filename = "ignition-gazebo-odometry-publisher-system">
-                <odom_frame>odom</odom_frame>
-                <robot_base_frame>${prefix}_base_link</robot_base_frame>
-                <odom_publish_frequency>60</odom_publish_frequency>
-                <odom_topic>odom</odom_topic>
-                <tf_topic>tf</tf_topic>
-                <publish_tf>true</publish_tf>
-                <dimensions>2</dimensions>
-            </plugin>
-            <!-- plugin for publishing the state of the joints -->
-            <plugin name = "ignition::gazebo::systems::JointStatePublisher" filename = "ignition-gazebo-joint-state-publisher-system">
-                <topic>joint_states</topic>
-                <joint_name>${prefix}_front_left_joint</joint_name>
-                <joint_name>${prefix}_front_right_joint</joint_name>
-                <joint_name>${prefix}_back_left_joint</joint_name>
-                <joint_name>${prefix}_back_right_joint</joint_name>
-            </plugin>
-        </gazebo>
-    </xacro:unless>
 </robot>
