Commit message: added in the sensor plugin, and added in the lidar plugin. wifi antennae are hit by the lidar rays, but we can just drop rays that have a value below the termination threshold

File: ros2_ws/src/agent_bringup/urdf/agent_gazebo_properties.xacro (robot description, xacro)
@@ -5,4 +5,5 @@
     <xacro:property name = "mu2" value = "0.1"/>
     <xacro:property name = "minDepth" value = "0.0001"/>
+    <xacro:property name = "piValue" value = "3.14159265359"/>
     <!-- LINK REFERENCES-->
     <gazebo reference = "${prefix}_front_right_wheel_link">
@@ -27,4 +28,31 @@
     </gazebo>
     <!-- PLUGINS -->
+    <!-- sensors plugin -->
+    <gazebo>
+        <plugin name = "ignition::gazebo::systems::Sensors" filename = "ignition-gazebo-sensors-system"/>
+    </gazebo>
+    <!-- lidar sensor -->
+    <gazebo reference = "${prefix}_lidar_link">
+        <sensor name = "laser" type = "gpu_lidar">
+            <pose>0 0 0.0093 0 0 0</pose>
+            <visualize>true</visualize>
+            <update_rate>10</update_rate>
+            <lidar>
+                <scan>
+                    <horizontal>
+                        <samples>1600</samples>
+                        <min_angle>${-piValue}</min_angle>
+                        <max_angle>${piValue}</max_angle>
+                    </horizontal>
+                </scan>
+                <range>
+                    <min>0.05</min>
+                    <max>12.0</max>
+                </range>
+            </lidar>
+            <topic>scan</topic>
+            <gz_frame_id>${prefix}_lidar_link</gz_frame_id>
+        </sensor>
+    </gazebo>
     <xacro:unless value = "$(arg use_ros_control)">
         <gazebo>

Commit message: added IMU to ``Gazebo``. this will be used to correct the yaw measurement provided by the ``/odom`` topic

File: ros2_ws/src/agent_bringup/urdf/agent_gazebo_properties.xacro (robot description, xacro)
@@ -59,3 +59,16 @@
         </sensor>
     </gazebo>
+    <!-- IMU plugin -->
+    <gazebo>
+        <plugin name = "ignition::gazebo::systems::Imu" filename = "ignition-gazebo-imu-system"/>
+    </gazebo>
+    <!-- IMU sensor -->
+    <gazebo reference = "${prefix}_imu_link">
+        <sensor name = "imu_sensor" type = "imu">
+            <always_on>1</always_on>
+            <update_rate>50</update_rate>
+            <visualize>true</visualize>
+            <topic>imu_data</topic>
+        </sensor>
+    </gazebo>
 </robot>

File: ros2_ws/src/agent_bringup/urdf/agent_peripherals.xacro (robot description, xacro)
@@ -66,3 +66,18 @@
         <child link = "${prefix}_depth_camera_optical_link"/>
     </joint>
+    <!-- IMU -->
+    <link name = "${prefix}_imu_link">
+        <inertial>
+            <mass value = "0.01"/>
+            <origin xyz = "0 0 0" rpy = "0 0 0"/>
+            <inertia ixx = "1e-6" iyy = "1e-6" izz = "1e-6"
+                     ixy = "0"    ixz = "0"    iyz = "0"/>
+        </inertial>
+    </link>
+    <!-- IMU to chassis joint -->
+    <joint name = "${prefix}_imu_chassis_joint" type = "fixed">
+        <origin xyz = "0 0 0" rpy = "0 0 0"/>
+        <parent link = "${prefix}_chassis_link"/>
+        <child link = "${prefix}_imu_link"/>
+    </joint>
 </robot>
