Commit message: fixed issues with URDF, namely missing a xacro property and legacy path name

File: ros2_ws/src/agent_bringup/urdf/agent_body.xacro (robot description, xacro)
@@ -2,4 +2,5 @@
 <robot xmlns:xacro = "http://www.ros.org/wiki/xacro">
     <!-- PROPERTIES -->
+    <xacro:property name = "a" value = "1.0"/>          <!-- scalar used for inertia-->
     <xacro:property name = "d" value = "1.0"/>          <!-- scalar used for damping -->
     <xacro:property name = "o" value = "0.0"/>          <!-- tuneable offset for wheel collision -->

File: ros2_ws/src/agent_bringup/urdf/agent_peripherals.xacro (robot description, xacro)
@@ -7,5 +7,5 @@
             <origin xyz = "0 0 0" rpy = "1.570796 0 1.570796"/>
             <geometry>
-                <mesh filename = "file://$(find mrs_robot_launcher)/meshes/lidar.STL" scale = "0.001 0.001 0.001"/>
+                <mesh filename = "file://$(find agent_bringup)/meshes/lidar.STL" scale = "0.001 0.001 0.001"/>
             </geometry>
             <material name = "black"/>

Commit message: changes to visual appearance of agent

File: ros2_ws/src/agent_bringup/urdf/agent_body.xacro (robot description, xacro)
@@ -13,4 +13,7 @@
     <material name = "gray">
         <color rgba = "0.83 0.83 0.83 1"/>
+    </material>
+    <material name = "green">
+        <color rgba = "0 1 0 1"/>
     </material>
     <!-- MACROS -->
@@ -46,5 +49,5 @@
                 <mesh filename = "file://$(find agent_bringup)/meshes/chassis.STL"/>
             </geometry>
-            <material name = "black"/>
+            <material name = "green"/>
         </visual>
         <collision>
@@ -77,5 +80,5 @@
                 <mesh filename = "file://$(find agent_bringup)/meshes/front_right_wheel.STL"/>
             </geometry>
-            <material name = "black"/>
+            <material name = "gray"/>
         </visual>
         <collision>
@@ -109,5 +112,5 @@
                 <mesh filename = "file://$(find agent_bringup)/meshes/front_left_wheel.STL"/>
             </geometry>
-            <material name = "black"/>
+            <material name = "gray"/>
         </visual>
         <collision>
@@ -141,5 +144,5 @@
                 <mesh filename = "file://$(find agent_bringup)/meshes/back_right_wheel.STL"/>
             </geometry>
-            <material name = "black"/>
+            <material name = "gray"/>
         </visual>
         <collision>
@@ -173,5 +176,5 @@
                 <mesh filename = "file://$(find agent_bringup)/meshes/back_left_wheel.STL"/>
             </geometry>
-            <material name = "black"/>
+            <material name = "gray"/>
         </visual>
         <collision>

Commit message: added limits to joints

File: ros2_ws/src/agent_bringup/urdf/agent_body.xacro (robot description, xacro)
@@ -86,4 +86,5 @@
             <geometry>
                 <cylinder radius = "0.0325" length = "0.03035"/>
+                <!-- <sphere radius = "0.0325"/> -->
             </geometry>
         </collision>
@@ -104,4 +105,5 @@
         <axis xyz = "0 1 0" rpy = "0 0 0"/>
         <dynamics damping = "${d}"/>
+        <limit effort = "0.05" velocity = "10.0"/>
     </joint>
     <!-- front left wheel link -->
@@ -118,4 +120,5 @@
             <geometry>
                 <cylinder radius = "0.0325" length = "0.03035"/>
+                <!-- <sphere radius = "0.0325"/> -->
             </geometry>
         </collision>
@@ -136,4 +139,5 @@
         <axis xyz = "0 1 0" rpy = "0 0 0"/>
         <dynamics damping = "${d}"/>
+        <limit effort = "0.05" velocity = "10.0"/>
     </joint>
     <!-- back right wheel link -->
@@ -150,4 +154,5 @@
             <geometry>
                 <cylinder radius = "0.0325" length = "0.03035"/>
+                <!-- <sphere radius = "0.0325"/> -->
             </geometry>
         </collision>
@@ -168,4 +173,5 @@
         <axis xyz = "0 1 0" rpy = "0 0 0"/>
         <dynamics damping = "${d}"/>
+        <limit effort = "0.05" velocity = "10.0"/>
     </joint>
     <!-- back left wheel link -->
@@ -182,4 +188,5 @@
             <geometry>
                 <cylinder radius = "0.0325" length = "0.03035"/>
+                <!-- <sphere radius = "0.0325"/> -->
             </geometry>
         </collision>
@@ -200,4 +207,5 @@
         <axis xyz = "0 1 0" rpy = "0 0 0"/>
         <dynamics damping = "${d}"/>
+        <limit effort = "0.05" velocity = "10.0"/>
     </joint>
 </robot>

Commit message: create xacro macros, modify gazebo LiDAR, and more controller yaml configurations
created macros to reduce rewritten code in the xacro files and faster prototyping

agent_body.xacro:
- wheel_link macro
- wheel_joint macro

agent_gazebo_properties.xacro
- wheel_link xacro to add gazebo properties to the wheel links
- increase the minimum LiDAR range to drop the antennae readings (might need reconsideration)
- change the LiDAR range from (-pi,pi) to (0,2pi) to match the MuJoCo DRL training observation

agent_ros_control.xacro
- make a xacro macro for ros2 control command and state interface of the joints+

File: ros2_ws/src/agent_bringup/urdf/agent_body.xacro (robot description, xacro)
@@ -7,4 +7,6 @@
     <xacro:property name = "c_mass" value = "2.415"/>   <!-- chassis mass in kg -->
     <xacro:property name = "w_mass" value = "0.058"/>   <!-- wheel mass in kg -->
+    <xacro:property name = "wheel_effort" value = "0.5"/>
+    <xacro:property name = "wheel_max_vel" value = "10.0"/>
     <!-- MATERIALS -->
     <material name = "black">
@@ -37,4 +39,42 @@
             izz = "${a * mass * (w**2 + d**2) / 12}"
         />
+    </xacro:macro>
+    <xacro:macro name = "wheel_link" params = "prefix position">
+        <!-- position is one of front_right, front_left, back_right, back_left-->
+        <link name = "${prefix}_${position}_wheel_link">
+            <visual>
+                <origin xyz = "0 0 0" rpy = "1.570796 0 0"/>
+                <geometry>
+                    <mesh filename = "file://$(find agent_bringup)/meshes/${position}_wheel.STL"/>
+                </geometry>
+                <material name = "gray"/>
+            </visual>
+            <collision>
+                <origin xyz = "0 0 ${-o}" rpy = "1.570796 0 0"/>
+                <geometry>
+                    <!-- <cylinder radius = "0.0325" length = "0.03035"/> -->
+                    <sphere radius = "0.0325"/>
+                </geometry>
+            </collision>
+            <inertial>
+                <mass value = "${w_mass}"/>
+                <xacro:cylinder_inertia
+                    mass = "${w_mass}"
+                    radius = "0.0325"
+                    length = "0.03035"
+                />
+            </inertial>
+        </link>
+    </xacro:macro>
+    <xacro:macro name = "wheel_joint" params = "prefix position xyz">
+        <!-- position is one of front_right, front_left, back_right, back_left-->
+        <joint name="${prefix}_${position}_joint" type="continuous">
+            <origin xyz = "${xyz}" rpy = "0 0 0"/>
+            <parent link = "${prefix}_chassis_link"/>
+            <child link = "${prefix}_${position}_wheel_link"/>
+            <axis xyz = "0 1 0" rpy = "0 0 0"/>
+            <dynamics damping = "${d}"/>
+            <limit effort = "${wheel_effort}" velocity = "${wheel_max_vel}"/>
+        </joint>
     </xacro:macro>
     <!-- START -->
@@ -73,139 +113,11 @@
         <origin xyz = "0 0 0.07115" rpy = "0 0 0"/> <!-- origin offset of 0.07115 -->
     </joint>
-    <!-- front right wheel link -->
-    <link name = "${prefix}_front_right_wheel_link">
-        <visual>
-            <origin xyz = "0 0 0" rpy = "1.570796 0 0"/>
-            <geometry>
-                <mesh filename = "file://$(find agent_bringup)/meshes/front_right_wheel.STL"/>
-            </geometry>
-            <material name = "gray"/>
-        </visual>
-        <collision>
-            <origin xyz = "0 0 ${-o}" rpy = "1.570796 0 0"/>
-            <geometry>
-                <!-- <cylinder radius = "0.0325" length = "0.03035"/> -->
-                <sphere radius = "0.0325"/>
-            </geometry>
-        </collision>
-        <inertial>
-            <mass value = "${w_mass}"/>
-            <xacro:cylinder_inertia
-                mass = "${w_mass}"
-                radius = "0.0325"
-                length = "0.03035"
-            />
-        </inertial>
-    </link>
-    <!-- front right wheel to chassis joint -->
-    <joint name = "${prefix}_front_right_joint" type = "continuous">
-        <origin xyz = "0.08 -0.08475 -0.0389" rpy = "0 0 0"/>
-        <parent link = "${prefix}_chassis_link"/>
-        <child link = "${prefix}_front_right_wheel_link"/>
-        <axis xyz = "0 1 0" rpy = "0 0 0"/>
-        <dynamics damping = "${d}"/>
-        <limit effort = "0.05" velocity = "10.0"/>
-    </joint>
-    <!-- front left wheel link -->
-    <link name = "${prefix}_front_left_wheel_link">
-        <visual>
-            <origin xyz = "0 0 0" rpy = "1.570796 0 0"/>
-            <geometry>
-                <mesh filename = "file://$(find agent_bringup)/meshes/front_left_wheel.STL"/>
-            </geometry>
-            <material name = "gray"/>
-        </visual>
-        <collision>
-            <origin xyz = "0 0 ${-o}" rpy = "1.570796 0 0"/>
-            <geometry>
-                <!-- <cylinder radius = "0.0325" length = "0.03035"/> -->
-                <sphere radius = "0.0325"/>
-            </geometry>
-        </collision>
-        <inertial>
-            <mass value = "${w_mass}"/>
-            <xacro:cylinder_inertia
-                mass = "${w_mass}"
-                radius = "0.0325"
-                length = "0.03035"
-            />
-        </inertial>
-    </link>
-    <!-- front left wheel to chassis joint -->
-    <joint name = "${prefix}_front_left_joint" type = "continuous">
-        <origin xyz = "0.08 0.08475 -0.0389" rpy = "0 0 0"/>
-        <parent link = "${prefix}_chassis_link"/>
-        <child link = "${prefix}_front_left_wheel_link"/>
-        <axis xyz = "0 1 0" rpy = "0 0 0"/>
-        <dynamics damping = "${d}"/>
-        <limit effort = "0.05" velocity = "10.0"/>
-    </joint>
-    <!-- back right wheel link -->
-    <link name = "${prefix}_back_right_wheel_link">
-        <visual>
-            <origin xyz = "0 0 0" rpy = "1.570796 0 0"/>
-            <geometry>
-                <mesh filename = "file://$(find agent_bringup)/meshes/back_right_wheel.STL"/>
-            </geometry>
-            <material name = "gray"/>
-        </visual>
-        <collision>
-            <origin xyz = "0 0 ${-o}" rpy = "1.570796 0 0"/>
-            <geometry>
-                <!-- <cylinder radius = "0.0325" length = "0.03035"/> -->
-                <sphere radius = "0.0325"/>
-            </geometry>
-        </collision>
-        <inertial>
-            <mass value = "${w_mass}"/>
-            <xacro:cylinder_inertia
-                mass = "${w_mass}"
-                radius = "0.0325"
-                length = "0.03035"
-            />
-        </inertial>
-    </link>
-    <!-- back right wheel to chassis joint -->
-    <joint name = "${prefix}_back_right_joint" type = "continuous">
-        <origin xyz = "-0.08 -0.08475 -0.0389" rpy = "0 0 0"/>   <!-- z was -0.03946 -->
-        <parent link = "${prefix}_chassis_link"/>
-        <child link = "${prefix}_back_right_wheel_link"/>
-        <axis xyz = "0 1 0" rpy = "0 0 0"/>
-        <dynamics damping = "${d}"/>
-        <limit effort = "0.05" velocity = "10.0"/>
-    </joint>
-    <!-- back left wheel link -->
-    <link name = "${prefix}_back_left_wheel_link">
-        <visual>
-            <origin xyz = "0 0 0" rpy = "1.570796 0 0"/>
-            <geometry>
-                <mesh filename = "file://$(find agent_bringup)/meshes/back_left_wheel.STL"/>
-            </geometry>
-            <material name = "gray"/>
-        </visual>
-        <collision>
-            <origin xyz = "0 0 ${-o}" rpy = "1.570796 0 0"/>
-            <geometry>
-                <!-- <cylinder radius = "0.0325" length = "0.03035"/> -->
-                <sphere radius = "0.0325"/>
-            </geometry>
-        </collision>
-        <inertial>
-            <mass value = "${w_mass}"/>
-            <xacro:cylinder_inertia
-                mass = "${w_mass}"
-                radius = "0.0325"
-                length = "0.03035"
-            />
-        </inertial>
-    </link>
-    <!-- back left wheel to chassis joint -->
-    <joint name = "${prefix}_back_left_joint" type = "continuous">
-        <origin xyz = "-0.08 0.08475 -0.0389" rpy = "0 0 0"/> <!-- z was -0.03954 -->
-        <parent link = "${prefix}_chassis_link"/>
-        <child link = "${prefix}_back_left_wheel_link"/>
-        <axis xyz = "0 1 0" rpy = "0 0 0"/>
-        <dynamics damping = "${d}"/>
-        <limit effort = "0.05" velocity = "10.0"/>
-    </joint>
+    <xacro:wheel_link prefix="${prefix}" position="front_right"/>
+    <xacro:wheel_joint prefix="${prefix}" position="front_right" xyz="0.08 -0.08475 -0.0389"/>
+    <xacro:wheel_link prefix="${prefix}" position="front_left"/>
+    <xacro:wheel_joint prefix="${prefix}" position="front_left" xyz="0.08 0.08475 -0.0389"/>
+    <xacro:wheel_link prefix="${prefix}" position="back_right"/>
+    <xacro:wheel_joint prefix="${prefix}" position="back_right" xyz="-0.08 -0.08475 -0.0389"/>
+    <xacro:wheel_link prefix="${prefix}" position="back_left"/>
+    <xacro:wheel_joint prefix="${prefix}" position="back_left" xyz="-0.08 0.08475 -0.0389"/>
 </robot>

File: ros2_ws/src/agent_bringup/urdf/agent_gazebo_properties.xacro (robot description, xacro)
@@ -2,33 +2,22 @@
 <robot xmlns:xacro = "http://www.ros.org/wiki/xacro">
     <!-- PROPERTIES -->
-    <xacro:property name = "mu1" value = "0.50"/>
-    <xacro:property name = "mu2" value = "0.01"/>
+    <xacro:property name = "mu1" value = "1.00"/>
+    <xacro:property name = "mu2" value = "0.03"/>
     <xacro:property name = "minDepth" value = "0.0001"/>
     <xacro:property name = "piValue" value = "3.14159265359"/>
+    <!-- MACROS -->
+    <xacro:macro name = "wheel_link" params = "position">
+        <gazebo reference = "${prefix}_${position}_wheel_link">
+            <mu1 value = "${mu1}"/>
+            <mu2 value = "${mu2}"/>
+            <fdir1>1 0 0</fdir1>
+            <minDepth value = "${minDepth}"/>
+        </gazebo>
+    </xacro:macro>
     <!-- LINK REFERENCES-->
-    <gazebo reference = "${prefix}_front_right_wheel_link">
-        <mu1 value = "${mu1}"/>
-        <mu2 value = "${mu2}"/>
-        <fdir1>1 0 0</fdir1>
-        <minDepth value = "${minDepth}"/>
-    </gazebo>
-    <gazebo reference = "${prefix}_front_left_wheel_link">
-        <mu1 value = "${mu1}"/>
-        <mu2 value = "${mu2}"/>
-        <fdir1>1 0 0</fdir1>
-        <minDepth value = "${minDepth}"/>
-    </gazebo>
-    <gazebo reference = "${prefix}_back_right_wheel_link">
-        <mu1 value = "${mu1}"/>
-        <mu2 value = "${mu2}"/>
-        <fdir1>1 0 0</fdir1>
-        <minDepth value = "${minDepth}"/>
-    </gazebo>
-    <gazebo reference = "${prefix}_back_left_wheel_link">
-        <mu1 value = "${mu1}"/>
-        <mu2 value = "${mu2}"/>
-        <fdir1>1 0 0</fdir1>
-        <minDepth value = "${minDepth}"/>
-    </gazebo>
+    <xacro:wheel_link position="front_right"/>
+    <xacro:wheel_link position="front_left"/>
+    <xacro:wheel_link position="back_right"/>
+    <xacro:wheel_link position="back_left"/>
     <!-- PLUGINS -->
     <!-- sensors plugin -->
@@ -46,10 +35,10 @@
                     <horizontal>
                         <samples>1600</samples>
-                        <min_angle>${-piValue}</min_angle>
-                        <max_angle>${piValue}</max_angle>
+                        <min_angle>0.0</min_angle>
+                        <max_angle>${2 * piValue}</max_angle>
                     </horizontal>
                 </scan>
                 <range>
-                    <min>0.05</min>
+                    <min>0.15</min>
                     <max>12.0</max>
                 </range>

File: ros2_ws/src/agent_bringup/urdf/agent_ros_control.xacro (robot description, xacro)
@@ -1,10 +1,6 @@
 <?xml version = "1.0"?>
 <robot xmlns:xacro = "http://www.ros.org/wiki/xacro">
-    <!-- instantiate the system -->
-    <ros2_control name = "GazeboSystem" type = "system">
-        <hardware>
-            <plugin>gz_ros2_control/GazeboSimSystem</plugin>
-        </hardware>
-        <joint name = "${prefix}_front_left_joint">
+    <xacro:macro name = "wheel_joint_control" params = "position">
+        <joint name="${prefix}_${position}_joint">
             <command_interface name = "velocity">
                 <param name = "min">0.0</param>
@@ -14,28 +10,14 @@
             <state_interface name="position"/>
         </joint>
-        <joint name = "${prefix}_front_right_joint">
-            <command_interface name = "velocity">
-                <param name = "min">0.0</param>
-                <param name = "max">10.0</param>
-            </command_interface>
-            <state_interface name="velocity"/>
-            <state_interface name="position"/>
-        </joint>
-        <joint name = "${prefix}_back_left_joint">
-            <command_interface name = "velocity">
-                <param name = "min">0.0</param>
-                <param name = "max">10.0</param>
-            </command_interface>
-            <state_interface name="velocity"/>
-            <state_interface name="position"/>
-        </joint>
-        <joint name = "${prefix}_back_right_joint">
-            <command_interface name = "velocity">
-                <param name = "min">0.0</param>
-                <param name = "max">10.0</param>
-            </command_interface>
-            <state_interface name="velocity"/>
-            <state_interface name="position"/>
-        </joint>
+    </xacro:macro>
+    <!-- instantiate the system -->
+    <ros2_control name = "GazeboSystem" type = "system">
+        <hardware>
+            <plugin>gz_ros2_control/GazeboSimSystem</plugin>
+        </hardware>
+        <xacro:wheel_joint_control position="front_right"/>
+        <xacro:wheel_joint_control position="front_left"/>
+        <xacro:wheel_joint_control position="back_right"/>
+        <xacro:wheel_joint_control position="back_left"/>
     </ros2_control>
     <gazebo>

Commit message: modify EKF fusion and (co)variance) + Gazebo property changes (wheel vel + LiDAR angle range)
- removed yaw and ay estimation from wheel odometry
- used linear x + y velocities of lidar odom in EKF fusion improved the odometry and addressed the jumpy update after a long command pause
- removed ax fusion from IMU

- increased max wheel vel from 10.0 to 30.0
- increased mu2
- changed the LiDAR min-max angle range

- tuned covariance to make lidar_odom's pose and twist covariance tighter

File: ros2_ws/src/agent_bringup/urdf/agent_body.xacro (robot description, xacro)
@@ -8,5 +8,5 @@
     <xacro:property name = "w_mass" value = "0.058"/>   <!-- wheel mass in kg -->
     <xacro:property name = "wheel_effort" value = "0.5"/>
-    <xacro:property name = "wheel_max_vel" value = "10.0"/>
+    <xacro:property name = "wheel_max_vel" value = "30.0"/>
     <!-- MATERIALS -->
     <material name = "black">

File: ros2_ws/src/agent_bringup/urdf/agent_gazebo_properties.xacro (robot description, xacro)
@@ -2,6 +2,6 @@
 <robot xmlns:xacro = "http://www.ros.org/wiki/xacro">
     <!-- PROPERTIES -->
-    <xacro:property name = "mu1" value = "1.00"/>
-    <xacro:property name = "mu2" value = "0.03"/>
+    <xacro:property name = "mu1" value = "1.0"/>
+    <xacro:property name = "mu2" value = "0.1"/>
     <xacro:property name = "minDepth" value = "0.0001"/>
     <xacro:property name = "piValue" value = "3.14159265359"/>
@@ -35,6 +35,6 @@
                     <horizontal>
                         <samples>1600</samples>
-                        <min_angle>0.0</min_angle>
-                        <max_angle>${2 * piValue}</max_angle>
+                        <min_angle>${-piValue}</min_angle>
+                        <max_angle>${piValue}</max_angle>
                     </horizontal>
                 </scan>

File: ros2_ws/src/agent_bringup/urdf/agent_ros_control.xacro (robot description, xacro)
@@ -5,5 +5,5 @@
             <command_interface name = "velocity">
                 <param name = "min">0.0</param>
-                <param name = "max">10.0</param>
+                <param name = "max">30.0</param>
             </command_interface>
             <state_interface name="velocity"/>

Commit message: adjust the LiDAR obs in policy_node + misc changes
- increased maximum wheel vel from 30 to 50
- reduced the LiDAR min range since I modified how the LiDAR rays hitting the antennae are handled

in policy_node
- handle the TD3/SAC loading and inferencing, so it is now as easy as specifying the name and the rest is automated
- increase ctrl frequency to match that of MuJoCo (might be unneccesary)
- modified LiDAR sensor processing (and made the policy worked in DRL)

File: ros2_ws/src/agent_bringup/urdf/agent_body.xacro (robot description, xacro)
@@ -8,5 +8,5 @@
     <xacro:property name = "w_mass" value = "0.058"/>   <!-- wheel mass in kg -->
     <xacro:property name = "wheel_effort" value = "0.5"/>
-    <xacro:property name = "wheel_max_vel" value = "30.0"/>
+    <xacro:property name = "wheel_max_vel" value = "50.0"/>
     <!-- MATERIALS -->
     <material name = "black">

File: ros2_ws/src/agent_bringup/urdf/agent_gazebo_properties.xacro (robot description, xacro)
@@ -3,5 +3,5 @@
     <!-- PROPERTIES -->
     <xacro:property name = "mu1" value = "1.0"/>
-    <xacro:property name = "mu2" value = "0.1"/>
+    <xacro:property name = "mu2" value = "0.3"/>
     <xacro:property name = "minDepth" value = "0.0001"/>
     <xacro:property name = "piValue" value = "3.14159265359"/>
@@ -40,5 +40,5 @@
                 </scan>
                 <range>
-                    <min>0.15</min>
+                    <min>0.13</min>
                     <max>12.0</max>
                 </range>

File: ros2_ws/src/agent_bringup/urdf/agent_ros_control.xacro (robot description, xacro)
@@ -5,5 +5,5 @@
             <command_interface name = "velocity">
                 <param name = "min">0.0</param>
-                <param name = "max">30.0</param>
+                <param name = "max">50.0</param>
             </command_interface>
             <state_interface name="velocity"/>
